File: CircuitDesing/embebidos/Potencia.kicad_sch (KiCad schematic)
At the start: 0 parts

Commit message: Potencia
Primera propuesta del esquema de potencia
Parts:
- added C4: (no value), symbol Device:C_Polarized
- added D? (x4): 1N5822, Diode_THT:D_DO-201AD_P15.24mm_Horizontal, symbol Diode:1N5822
Connections:
- new net GND: C4.2, D?.2 (A), D?.2 (A)
- new net Tap_1: D?.1 (K), D?.2 (A)
- new net Tap_2: D?.1 (K), D?.2 (A)
- new net out_rect: C4.1, D?.1 (K), D?.1 (K)
Other:
- added sheet Buck (Buck-converter_sch.kicad_sch)
- added sheet LDO (untitled.kicad_sch)
Changed lines of the file:
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@@
 (kicad_sch (version 20211123) (generator eeschema)
   (paper "A4")
+  (junction (at 115.57 50.8) (diameter 0) (color 0 0 0 0)
+  )
+  (junction (at 78.74 85.09) (diameter 0) (color 0 0 0 0)
+  )
+  (junction (at 86.36 50.8) (diameter 0) (color 0 0 0 0)
+  )
+  (junction (at 86.36 69.85) (diameter 0) (color 0 0 0 0)
+  )
+  (junction (at 86.36 85.09) (diameter 0) (color 0 0 0 0)
+  )
+  (junction (at 67.31 66.04) (diameter 0) (color 0 0 0 0)
+  )
+  (wire (pts (xy 86.36 50.8) (xy 86.36 54.61))
+    (stroke (width 0) (type default) (color 0 0 0 0))
+  )
+  (wire (pts (xy 166.37 57.15) (xy 170.18 57.15))
+    (stroke (width 0) (type default) (color 0 0 0 0))
+  )
+  (wire (pts (xy 86.36 69.85) (xy 86.36 71.12))
+    (stroke (width 0) (type default) (color 0 0 0 0))
+  )
+  (wire (pts (xy 86.36 78.74) (xy 86.36 85.09))
+    (stroke (width 0) (type default) (color 0 0 0 0))
+  )
+  (wire (pts (xy 67.31 62.23) (xy 67.31 66.04))
+    (stroke (width 0) (type default) (color 0 0 0 0))
+  )
+  (wire (pts (xy 86.36 85.09) (xy 78.74 85.09))
+    (stroke (width 0) (type default) (color 0 0 0 0))
+  )
+  (wire (pts (xy 215.9 99.06) (xy 220.98 99.06))
+    (stroke (width 0) (type default) (color 0 0 0 0))
+  )
+  (wire (pts (xy 62.23 69.85) (xy 86.36 69.85))
+    (stroke (width 0) (type default) (color 0 0 0 0))
+  )
+  (wire (pts (xy 115.57 85.09) (xy 86.36 85.09))
+    (stroke (width 0) (type default) (color 0 0 0 0))
+  )
+  (wire (pts (xy 115.57 62.23) (xy 115.57 50.8))
+    (stroke (width 0) (type default) (color 0 0 0 0))
+  )
+  (wire (pts (xy 215.9 57.15) (xy 220.98 57.15))
+    (stroke (width 0) (type default) (color 0 0 0 0))
+  )
+  (wire (pts (xy 67.31 54.61) (xy 67.31 50.8))
+    (stroke (width 0) (type default) (color 0 0 0 0))
+  )
+  (wire (pts (xy 115.57 69.85) (xy 115.57 85.09))
+    (stroke (width 0) (type default) (color 0 0 0 0))
+  )
+  (wire (pts (xy 166.37 99.06) (xy 170.18 99.06))
+    (stroke (width 0) (type default) (color 0 0 0 0))
+  )
+  (wire (pts (xy 67.31 50.8) (xy 86.36 50.8))
+    (stroke (width 0) (type default) (color 0 0 0 0))
+  )
+  (wire (pts (xy 62.23 72.39) (xy 62.23 69.85))
+    (stroke (width 0) (type default) (color 0 0 0 0))
+  )
+  (wire (pts (xy 67.31 66.04) (xy 67.31 71.12))
+    (stroke (width 0) (type default) (color 0 0 0 0))
+  )
+  (wire (pts (xy 78.74 85.09) (xy 67.31 85.09))
+    (stroke (width 0) (type default) (color 0 0 0 0))
+  )
+  (wire (pts (xy 52.07 66.04) (xy 67.31 66.04))
+    (stroke (width 0) (type default) (color 0 0 0 0))
+  )
+  (wire (pts (xy 52.07 72.39) (xy 62.23 72.39))
+    (stroke (width 0) (type default) (color 0 0 0 0))
+  )
+  (wire (pts (xy 86.36 62.23) (xy 86.36 69.85))
+    (stroke (width 0) (type default) (color 0 0 0 0))
+  )
+  (wire (pts (xy 115.57 50.8) (xy 120.65 50.8))
+    (stroke (width 0) (type default) (color 0 0 0 0))
+  )
+  (wire (pts (xy 67.31 78.74) (xy 67.31 85.09))
+    (stroke (width 0) (type default) (color 0 0 0 0))
+  )
+  (wire (pts (xy 115.57 50.8) (xy 86.36 50.8))
+    (stroke (width 0) (type default) (color 0 0 0 0))
+  )
+  (label "out_rect" (at 166.37 99.06 180)
+    (effects (font (size 1.27 1.27)) (justify right bottom))
+  )
+  (label "out_rect" (at 120.65 50.8 0)
+    (effects (font (size 1.27 1.27)) (justify left bottom))
+  )
+  (label "out_rect" (at 166.37 57.15 180)
+    (effects (font (size 1.27 1.27)) (justify right bottom))
+  )
+  (hierarchical_label "out_3.3v" (shape output) (at 220.98 99.06 0)
+    (effects (font (size 1.27 1.27)) (justify left))
+  )
+  (hierarchical_label "Tap_1" (shape input) (at 52.07 66.04 180)
+    (effects (font (size 1.27 1.27)) (justify right))
+  )
+  (hierarchical_label "out_5v" (shape output) (at 220.98 57.15 0)
+    (effects (font (size 1.27 1.27)) (justify left))
+  )
+  (hierarchical_label "Tap_2" (shape input) (at 52.07 72.39 180)
+    (effects (font (size 1.27 1.27)) (justify right))
+  )
+  (symbol (lib_id "Device:C_Polarized") (at 115.57 66.04 0) (unit 1)
+    (in_bom yes) (on_board yes) (fields_autoplaced)
+    (property "Reference" "C4" (id 0) (at 119.38 63.8809 0)
+      (effects (font (size 1.27 1.27)) (justify left))
+    )
+    (property "Value" "" (id 1) (at 119.38 66.4209 0)
+      (effects (font (size 1.27 1.27)) (justify left))
+    )
+    (property "Footprint" "" (id 2) (at 116.5352 69.85 0)
+      (effects (font (size 1.27 1.27)) hide)
+    )
+    (property "Datasheet" "~" (id 3) (at 115.57 66.04 0)
+      (effects (font (size 1.27 1.27)) hide)
+    )
+    (pin "1")
+    (pin "2")
+  )
+  (symbol (lib_id "Diode:1N5822") (at 86.36 74.93 270) (unit 1)
+    (in_bom yes) (on_board yes) (fields_autoplaced)
+    (property "Reference" "D?" (id 0) (at 88.9 73.3424 90)
+      (effects (font (size 1.27 1.27)) (justify left))
+    )
+    (property "Value" "1N5822" (id 1) (at 88.9 75.8824 90)
+      (effects (font (size 1.27 1.27)) (justify left))
+    )
+    (property "Footprint" "Diode_THT:D_DO-201AD_P15.24mm_Horizontal" (id 2) (at 81.915 74.93 0)
+      (effects (font (size 1.27 1.27)) hide)
+    )
+    (property "Datasheet" "http://www.vishay.com/docs/88526/1n5820.pdf" (id 3) (at 86.36 74.93 0)
+      (effects (font (size 1.27 1.27)) hide)
+    )
+    (pin "1")
+    (pin "2")
+  )
+  (symbol (lib_id "Diode:1N5822") (at 67.31 58.42 270) (unit 1)
+    (in_bom yes) (on_board yes) (fields_autoplaced)
+    (property "Reference" "D?" (id 0) (at 69.85 56.8324 90)
+      (effects (font (size 1.27 1.27)) (justify left))
+    )
+    (property "Value" "1N5822" (id 1) (at 69.85 59.3724 90)
+      (effects (font (size 1.27 1.27)) (justify left))
+    )
+    (property "Footprint" "Diode_THT:D_DO-201AD_P15.24mm_Horizontal" (id 2) (at 62.865 58.42 0)
+      (effects (font (size 1.27 1.27)) hide)
+    )
+    (property "Datasheet" "http://www.vishay.com/docs/88526/1n5820.pdf" (id 3) (at 67.31 58.42 0)
+      (effects (font (size 1.27 1.27)) hide)
+    )
+    (pin "1")
+    (pin "2")
+  )
+  (symbol (lib_id "power:GND") (at 78.74 85.09 0) (unit 1)
+    (in_bom yes) (on_board yes) (fields_autoplaced)
+    (property "Reference" "#PWR?" (id 0) (at 78.74 91.44 0)
+      (effects (font (size 1.27 1.27)) hide)
+    )
+    (property "Value" "GND" (id 1) (at 78.74 90.17 0))
+    (property "Footprint" "" (id 2) (at 78.74 85.09 0)
+      (effects (font (size 1.27 1.27)) hide)
+    )
+    (property "Datasheet" "" (id 3) (at 78.74 85.09 0)
+      (effects (font (size 1.27 1.27)) hide)
+    )
+    (pin "1")
+  )
+  (symbol (lib_id "Diode:1N5822") (at 67.31 74.93 270) (unit 1)
+    (in_bom yes) (on_board yes) (fields_autoplaced)
+    (property "Reference" "D?" (id 0) (at 69.85 73.3424 90)
+      (effects (font (size 1.27 1.27)) (justify left))
+    )
+    (property "Value" "1N5822" (id 1) (at 69.85 75.8824 90)
+      (effects (font (size 1.27 1.27)) (justify left))
+    )
+    (property "Footprint" "Diode_THT:D_DO-201AD_P15.24mm_Horizontal" (id 2) (at 62.865 74.93 0)
+      (effects (font (size 1.27 1.27)) hide)
+    )
+    (property "Datasheet" "http://www.vishay.com/docs/88526/1n5820.pdf" (id 3) (at 67.31 74.93 0)
+      (effects (font (size 1.27 1.27)) hide)
+    )
+    (pin "1")
+    (pin "2")
+  )
+  (symbol (lib_id "Diode:1N5822") (at 86.36 58.42 270) (unit 1)
+    (in_bom yes) (on_board yes) (fields_autoplaced)
+    (property "Reference" "D?" (id 0) (at 88.9 56.8324 90)
+      (effects (font (size 1.27 1.27)) (justify left))
+    )
+    (property "Value" "1N5822" (id 1) (at 88.9 59.3724 90)
+      (effects (font (size 1.27 1.27)) (justify left))
+    )
+    (property "Footprint" "Diode_THT:D_DO-201AD_P15.24mm_Horizontal" (id 2) (at 81.915 58.42 0)
+      (effects (font (size 1.27 1.27)) hide)
+    )
+    (property "Datasheet" "http://www.vishay.com/docs/88526/1n5820.pdf" (id 3) (at 86.36 58.42 0)
+      (effects (font (size 1.27 1.27)) hide)
+    )
+    (pin "1")
+    (pin "2")
+  )
+  (sheet (at 170.18 90.17) (size 45.72 21.59) (fields_autoplaced)
+    (stroke (width 0.1524) (type solid) (color 0 0 0 0))
+    (fill (color 0 0 0 0.0000))
+    (property "Sheet name" "LDO" (id 0) (at 170.18 89.4584 0)
+      (effects (font (size 1.27 1.27)) (justify left bottom))
+    )
+    (property "Sheet file" "untitled.kicad_sch" (id 1) (at 170.18 112.3446 0)
+      (effects (font (size 1.27 1.27)) (justify left top))
+    )
+    (pin "Buck_in" input (at 170.18 99.06 180)
+      (effects (font (size 1.27 1.27)) (justify left))
+    )
+    (pin "Buck_out" output (at 215.9 99.06 0)
+      (effects (font (size 1.27 1.27)) (justify right))
+    )
+  )
+  (sheet (at 170.18 45.72) (size 45.72 21.59) (fields_autoplaced)
+    (stroke (width 0.1524) (type solid) (color 0 0 0 0))
+    (fill (color 0 0 0 0.0000))
+    (property "Sheet name" "Buck" (id 0) (at 170.18 45.0084 0)
+      (effects (font (size 1.27 1.27)) (justify left bottom))
+    )
+    (property "Sheet file" "Buck-converter_sch.kicad_sch" (id 1) (at 170.18 67.8946 0)
+      (effects (font (size 1.27 1.27)) (justify left top))
+    )
+    (pin "Buck_out" output (at 215.9 57.15 0)
+      (effects (font (size 1.27 1.27)) (justify right))
+    )
+    (pin "Buck_in" input (at 170.18 57.15 180)
+      (effects (font (size 1.27 1.27)) (justify left))
+    )
+  )
 )

Commit message: Bootoption enable sw
Parts:
- C4: value (none) -> 470u
Changed lines of the file:
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@@
       (effects (font (size 1.27 1.27)) (justify left))
     )
-    (property "Value" "" (id 1) (at 119.38 66.4209 0)
+    (property "Value" "470u" (id 1) (at 119.38 66.4209 0)
       (effects (font (size 1.27 1.27)) (justify left))
     )
