File: CircuitDesing/embebidos/Buck-converter_sch.kicad_sch (KiCad schematic)
At the start: 5 parts

Commit message: Bootoption enable sw
Parts:
- C?: value (none) -> C_Polarized
- D?: value (none) -> 1N5822; footprint (none) -> Diode_THT:D_DO-201AD_P15.24mm_Horizontal
- L?: value (none) -> L
- U?: value (none) -> LM2576S-5; footprint (none) -> Package_TO_SOT_SMD:TO-263-5_TabPin3
Changed lines of the file:
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@@
       (effects (font (size 1.27 1.27)) (justify left))
     )
-    (property "Value" "" (id 1) (at 146.05 89.8524 90)
+    (property "Value" "1N5822" (id 1) (at 146.05 89.8524 90)
       (effects (font (size 1.27 1.27)) (justify left))
     )
-    (property "Footprint" "" (id 2) (at 139.065 88.9 0)
+    (property "Footprint" "Diode_THT:D_DO-201AD_P15.24mm_Horizontal" (id 2) (at 139.065 88.9 0)
       (effects (font (size 1.27 1.27)) hide)
     )
@@
     (in_bom yes) (on_board yes) (fields_autoplaced)
     (property "Reference" "L?" (id 0) (at 154.94 74.93 90))
-    (property "Value" "" (id 1) (at 154.94 77.47 90))
+    (property "Value" "L" (id 1) (at 154.94 77.47 90))
     (property "Footprint" "" (id 2) (at 154.94 81.28 0)
       (effects (font (size 1.27 1.27)) hide)
@@
       (effects (font (size 1.27 1.27)) (justify left))
     )
-    (property "Value" "" (id 1) (at 91.44 85.4709 0)
+    (property "Value" "C_Polarized" (id 1) (at 91.44 85.4709 0)
       (effects (font (size 1.27 1.27)) (justify left))
     )
@@
     (in_bom yes) (on_board yes) (fields_autoplaced)
     (property "Reference" "U?" (id 0) (at 121.92 68.58 0))
-    (property "Value" "" (id 1) (at 121.92 71.12 0))
-    (property "Footprint" "" (id 2) (at 121.92 85.09 0)
+    (property "Value" "LM2576S-5" (id 1) (at 121.92 71.12 0))
+    (property "Footprint" "Package_TO_SOT_SMD:TO-263-5_TabPin3" (id 2) (at 121.92 85.09 0)
       (effects (font (size 1.27 1.27) italic) (justify left) hide)
     )
@@
       (effects (font (size 1.27 1.27)) hide)
     )
-    (property "Value" "" (id 1) (at 87.63 93.98 0))
+    (property "Value" "GND" (id 1) (at 87.63 93.98 0))
     (property "Footprint" "" (id 2) (at 87.63 88.9 0)
       (effects (font (size 1.27 1.27)) hide)

Commit message: LDR
Comparacion LDR
Parts:
- C? (x2): value C_Polarized -> (none)
- L?: value L -> (none)
Changed lines of the file:
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@@
   )
   (symbol (lib_id "Device:L") (at 154.94 81.28 90) (unit 1)
-    (in_bom yes) (on_board yes) (fields_autoplaced)
-    (property "Reference" "L?" (id 0) (at 154.94 74.93 90))
-    (property "Value" "L" (id 1) (at 154.94 77.47 90))
+    (in_bom yes) (on_board yes)
+    (property "Reference" "L?" (id 0) (at 154.94 82.55 90))
+    (property "Value" "" (id 1) (at 154.94 77.47 90))
     (property "Footprint" "" (id 2) (at 154.94 81.28 0)
       (effects (font (size 1.27 1.27)) hide)
@@
       (effects (font (size 1.27 1.27)) (justify left))
     )
-    (property "Value" "C_Polarized" (id 1) (at 91.44 85.4709 0)
+    (property "Value" "" (id 1) (at 91.44 85.4709 0)
       (effects (font (size 1.27 1.27)) (justify left))
     )
@@
       (effects (font (size 1.27 1.27)) (justify left))
     )
-    (property "Value" "C_Polarized" (id 1) (at 168.91 89.2809 0)
+    (property "Value" "" (id 1) (at 168.91 89.2809 0)
       (effects (font (size 1.27 1.27)) (justify left))
     )

Commit message: Sensor Ultrasonido
Parts:
- C?, L?: value (none) -> 100u
- C?: value (none) -> 1000u
Changed lines of the file:
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@@
     (in_bom yes) (on_board yes)
     (property "Reference" "L?" (id 0) (at 154.94 82.55 90))
-    (property "Value" "" (id 1) (at 154.94 77.47 90))
+    (property "Value" "100u" (id 1) (at 154.94 77.47 90))
     (property "Footprint" "" (id 2) (at 154.94 81.28 0)
       (effects (font (size 1.27 1.27)) hide)
@@
       (effects (font (size 1.27 1.27)) (justify left))
     )
-    (property "Value" "" (id 1) (at 91.44 85.4709 0)
+    (property "Value" "100u" (id 1) (at 91.44 85.4709 0)
       (effects (font (size 1.27 1.27)) (justify left))
     )
@@
       (effects (font (size 1.27 1.27)) (justify left))
     )
-    (property "Value" "" (id 1) (at 168.91 89.2809 0)
+    (property "Value" "1000u" (id 1) (at 168.91 89.2809 0)
       (effects (font (size 1.27 1.27)) (justify left))
     )

Commit message: Huellas parciales
Parts:
- C5, C6: renamed from C?; footprint (none) -> Capacitor_SMD:C_0603_1608Metric_Pad1.08x0.95mm_HandSolder
- gave numbers to parts that had none: 3
Changed lines of the file:
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@@
   (symbol (lib_id "power:GND") (at 113.03 91.44 0) (unit 1)
     (in_bom yes) (on_board yes) (fields_autoplaced)
-    (property "Reference" "#PWR?" (id 0) (at 113.03 97.79 0)
+    (property "Reference" "#PWR018" (id 0) (at 113.03 97.79 0)
       (effects (font (size 1.27 1.27)) hide)
     )
@@
   (symbol (lib_id "power:GND") (at 165.1 92.71 0) (unit 1)
     (in_bom yes) (on_board yes) (fields_autoplaced)
-    (property "Reference" "#PWR?" (id 0) (at 165.1 99.06 0)
+    (property "Reference" "#PWR020" (id 0) (at 165.1 99.06 0)
       (effects (font (size 1.27 1.27)) hide)
     )
@@
   (symbol (lib_id "Diode:1N5822") (at 143.51 88.9 270) (unit 1)
     (in_bom yes) (on_board yes) (fields_autoplaced)
-    (property "Reference" "D?" (id 0) (at 146.05 87.3124 90)
+    (property "Reference" "D5" (id 0) (at 146.05 87.3124 90)
       (effects (font (size 1.27 1.27)) (justify left))
     )
@@
   (symbol (lib_id "Device:L") (at 154.94 81.28 90) (unit 1)
     (in_bom yes) (on_board yes)
-    (property "Reference" "L?" (id 0) (at 154.94 82.55 90))
+    (property "Reference" "L1" (id 0) (at 154.94 82.55 90))
     (property "Value" "100u" (id 1) (at 154.94 77.47 90))
     (property "Footprint" "" (id 2) (at 154.94 81.28 0)
@@
   (symbol (lib_id "Device:C_Polarized") (at 87.63 85.09 0) (unit 1)
     (in_bom yes) (on_board yes) (fields_autoplaced)
-    (property "Reference" "C?" (id 0) (at 91.44 82.9309 0)
+    (property "Reference" "C5" (id 0) (at 91.44 82.9309 0)
       (effects (font (size 1.27 1.27)) (justify left))
     )
@@
       (effects (font (size 1.27 1.27)) (justify left))
     )
-    (property "Footprint" "" (id 2) (at 88.5952 88.9 0)
+    (property "Footprint" "Capacitor_SMD:C_0603_1608Metric_Pad1.08x0.95mm_HandSolder" (id 2) (at 88.5952 88.9 0)
       (effects (font (size 1.27 1.27)) hide)
     )
@@
   (symbol (lib_id "Regulator_Switching:LM2576S-5") (at 121.92 78.74 0) (unit 1)
     (in_bom yes) (on_board yes) (fields_autoplaced)
-    (property "Reference" "U?" (id 0) (at 121.92 68.58 0))
+    (property "Reference" "U2" (id 0) (at 121.92 68.58 0))
     (property "Value" "LM2576S-5" (id 1) (at 121.92 71.12 0))
     (property "Footprint" "Package_TO_SOT_SMD:TO-263-5_TabPin3" (id 2) (at 121.92 85.09 0)
@@
   (symbol (lib_id "Device:C_Polarized") (at 165.1 88.9 0) (unit 1)
     (in_bom yes) (on_board yes) (fields_autoplaced)
-    (property "Reference" "C?" (id 0) (at 168.91 86.7409 0)
+    (property "Reference" "C6" (id 0) (at 168.91 86.7409 0)
       (effects (font (size 1.27 1.27)) (justify left))
     )
@@
       (effects (font (size 1.27 1.27)) (justify left))
     )
-    (property "Footprint" "" (id 2) (at 166.0652 92.71 0)
+    (property "Footprint" "Capacitor_SMD:C_0603_1608Metric_Pad1.08x0.95mm_HandSolder" (id 2) (at 166.0652 92.71 0)
       (effects (font (size 1.27 1.27)) hide)
     )
@@
   (symbol (lib_id "power:GND") (at 143.51 92.71 0) (unit 1)
     (in_bom yes) (on_board yes) (fields_autoplaced)
-    (property "Reference" "#PWR?" (id 0) (at 143.51 99.06 0)
+    (property "Reference" "#PWR019" (id 0) (at 143.51 99.06 0)
       (effects (font (size 1.27 1.27)) hide)
     )
@@
   (symbol (lib_id "power:GND") (at 87.63 88.9 0) (unit 1)
     (in_bom yes) (on_board yes) (fields_autoplaced)
-    (property "Reference" "#PWR?" (id 0) (at 87.63 95.25 0)
+    (property "Reference" "#PWR017" (id 0) (at 87.63 95.25 0)
       (effects (font (size 1.27 1.27)) hide)
     )

Commit message: Todas las huellas
Parts:
- L1: footprint (none) -> Inductor_SMD:L_0603_1608Metric_Pad1.05x0.95mm_HandSolder
Changed lines of the file:
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@@
     (property "Reference" "L1" (id 0) (at 154.94 82.55 90))
     (property "Value" "100u" (id 1) (at 154.94 77.47 90))
-    (property "Footprint" "" (id 2) (at 154.94 81.28 0)
+    (property "Footprint" "Inductor_SMD:L_0603_1608Metric_Pad1.05x0.95mm_HandSolder" (id 2) (at 154.94 81.28 0)
       (effects (font (size 1.27 1.27)) hide)
     )
