File: CircuitDesing/embebidos/Con_digital.kicad_sch (KiCad schematic)
At the start: 6 parts

Commit message: Ruteo completo
Parts:
- gave numbers to parts that had none: 2
- renumbered R1 to R27, R2 to R28, R3 to R29, R4 to R30
Changed lines of the file:
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@@
   (symbol (lib_id "Device:R") (at 87.63 81.28 0) (unit 1)
     (in_bom yes) (on_board yes) (fields_autoplaced)
-    (property "Reference" "R2" (id 0) (at 90.17 80.0099 0)
+    (property "Reference" "R28" (id 0) (at 90.17 80.0099 0)
       (effects (font (size 1.27 1.27)) (justify left))
     )
@@
   (symbol (lib_id "Device:R") (at 143.51 81.28 0) (unit 1)
     (in_bom yes) (on_board yes) (fields_autoplaced)
-    (property "Reference" "R4" (id 0) (at 146.05 80.0099 0)
+    (property "Reference" "R30" (id 0) (at 146.05 80.0099 0)
       (effects (font (size 1.27 1.27)) (justify left))
     )
@@
   (symbol (lib_id "Device:R") (at 125.73 81.28 0) (unit 1)
     (in_bom yes) (on_board yes) (fields_autoplaced)
-    (property "Reference" "R3" (id 0) (at 128.27 80.0099 0)
+    (property "Reference" "R29" (id 0) (at 128.27 80.0099 0)
       (effects (font (size 1.27 1.27)) (justify left))
     )
@@
   (symbol (lib_id "Transistor_FET:BSS138") (at 78.74 91.44 270) (unit 1)
     (in_bom yes) (on_board yes) (fields_autoplaced)
-    (property "Reference" "Q?" (id 0) (at 78.74 99.06 90))
+    (property "Reference" "Q15" (id 0) (at 78.74 99.06 90))
     (property "Value" "BSS138" (id 1) (at 78.74 101.6 90))
     (property "Footprint" "Package_TO_SOT_SMD:SOT-23" (id 2) (at 76.835 96.52 0)
@@
   (symbol (lib_id "Transistor_FET:BSS138") (at 134.62 91.44 270) (unit 1)
     (in_bom yes) (on_board yes) (fields_autoplaced)
-    (property "Reference" "Q?" (id 0) (at 134.62 99.06 90))
+    (property "Reference" "Q16" (id 0) (at 134.62 99.06 90))
     (property "Value" "BSS138" (id 1) (at 134.62 101.6 90))
     (property "Footprint" "Package_TO_SOT_SMD:SOT-23" (id 2) (at 132.715 96.52 0)
@@
   (symbol (lib_id "Device:R") (at 69.85 81.28 0) (unit 1)
     (in_bom yes) (on_board yes) (fields_autoplaced)
-    (property "Reference" "R1" (id 0) (at 72.39 80.0099 0)
+    (property "Reference" "R27" (id 0) (at 72.39 80.0099 0)
       (effects (font (size 1.27 1.27)) (justify left))
     )
