File: CircuitDesing/embebidos/untitled.kicad_sch (KiCad schematic)
At the start: 3 parts

Commit message: Bootoption enable sw
Parts:
- C7: renamed from C5; value (none) -> 10u
- C8: renamed from C6; value (none) -> 100u
- U?: value (none) -> LM1117-3.3
Changed lines of the file:
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@@
       (effects (font (size 1.27 1.27)) hide)
     )
-    (property "Value" "" (id 1) (at 104.14 83.82 0))
+    (property "Value" "GND" (id 1) (at 104.14 83.82 0))
     (property "Footprint" "" (id 2) (at 104.14 78.74 0)
       (effects (font (size 1.27 1.27)) hide)
@@
   (symbol (lib_id "Device:C_Polarized") (at 120.65 76.2 0) (unit 1)
     (in_bom yes) (on_board yes) (fields_autoplaced)
-    (property "Reference" "C6" (id 0) (at 124.46 74.0409 0)
+    (property "Reference" "C8" (id 0) (at 124.46 74.0409 0)
       (effects (font (size 1.27 1.27)) (justify left))
     )
-    (property "Value" "" (id 1) (at 124.46 76.5809 0)
+    (property "Value" "100u" (id 1) (at 124.46 76.5809 0)
       (effects (font (size 1.27 1.27)) (justify left))
     )
@@
     (in_bom yes) (on_board yes) (fields_autoplaced)
     (property "Reference" "U?" (id 0) (at 104.14 58.42 0))
-    (property "Value" "" (id 1) (at 104.14 60.96 0))
+    (property "Value" "LM1117-3.3" (id 1) (at 104.14 60.96 0))
     (property "Footprint" "" (id 2) (at 104.14 66.04 0)
       (effects (font (size 1.27 1.27)) hide)
@@
   (symbol (lib_id "Device:C_Polarized") (at 85.09 76.2 0) (unit 1)
     (in_bom yes) (on_board yes) (fields_autoplaced)
-    (property "Reference" "C5" (id 0) (at 88.9 74.0409 0)
+    (property "Reference" "C7" (id 0) (at 88.9 74.0409 0)
       (effects (font (size 1.27 1.27)) (justify left))
     )
-    (property "Value" "" (id 1) (at 88.9 76.5809 0)
+    (property "Value" "10u" (id 1) (at 88.9 76.5809 0)
       (effects (font (size 1.27 1.27)) (justify left))
     )

Commit message: Huellas parciales
Parts:
- C7, C8: footprint (none) -> Capacitor_SMD:C_0603_1608Metric_Pad1.08x0.95mm_HandSolder
- gave numbers to parts that had none: 1
Changed lines of the file:
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@@
   (symbol (lib_id "power:GND") (at 104.14 78.74 0) (unit 1)
     (in_bom yes) (on_board yes) (fields_autoplaced)
-    (property "Reference" "#PWR?" (id 0) (at 104.14 85.09 0)
+    (property "Reference" "#PWR022" (id 0) (at 104.14 85.09 0)
       (effects (font (size 1.27 1.27)) hide)
     )
@@
       (effects (font (size 1.27 1.27)) (justify left))
     )
-    (property "Footprint" "" (id 2) (at 121.6152 80.01 0)
+    (property "Footprint" "Capacitor_SMD:C_0603_1608Metric_Pad1.08x0.95mm_HandSolder" (id 2) (at 121.6152 80.01 0)
       (effects (font (size 1.27 1.27)) hide)
     )
@@
   (symbol (lib_id "power:GND") (at 120.65 80.01 0) (unit 1)
     (in_bom yes) (on_board yes) (fields_autoplaced)
-    (property "Reference" "#PWR?" (id 0) (at 120.65 86.36 0)
+    (property "Reference" "#PWR023" (id 0) (at 120.65 86.36 0)
       (effects (font (size 1.27 1.27)) hide)
     )
@@
   (symbol (lib_id "Regulator_Linear:LM1117-3.3") (at 104.14 66.04 0) (unit 1)
     (in_bom yes) (on_board yes) (fields_autoplaced)
-    (property "Reference" "U?" (id 0) (at 104.14 58.42 0))
+    (property "Reference" "U3" (id 0) (at 104.14 58.42 0))
     (property "Value" "LM1117-3.3" (id 1) (at 104.14 60.96 0))
     (property "Footprint" "" (id 2) (at 104.14 66.04 0)
@@
   (symbol (lib_id "power:GND") (at 85.09 80.01 0) (unit 1)
     (in_bom yes) (on_board yes) (fields_autoplaced)
-    (property "Reference" "#PWR?" (id 0) (at 85.09 86.36 0)
+    (property "Reference" "#PWR021" (id 0) (at 85.09 86.36 0)
       (effects (font (size 1.27 1.27)) hide)
     )
@@
       (effects (font (size 1.27 1.27)) (justify left))
     )
-    (property "Footprint" "" (id 2) (at 86.0552 80.01 0)
+    (property "Footprint" "Capacitor_SMD:C_0603_1608Metric_Pad1.08x0.95mm_HandSolder" (id 2) (at 86.0552 80.01 0)
       (effects (font (size 1.27 1.27)) hide)
     )

Commit message: Todas las huellas
Parts:
- U3: footprint (none) -> Package_TO_SOT_THT:TO-220-3_Vertical
Changed lines of the file:
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@@
     (property "Reference" "U3" (id 0) (at 104.14 58.42 0))
     (property "Value" "LM1117-3.3" (id 1) (at 104.14 60.96 0))
-    (property "Footprint" "" (id 2) (at 104.14 66.04 0)
+    (property "Footprint" "Package_TO_SOT_THT:TO-220-3_Vertical" (id 2) (at 104.14 66.04 0)
       (effects (font (size 1.27 1.27)) hide)
     )

Commit message: Actualizacion huellas
Huellas+Programador
Parts:
- removed U3: LM1117-3.3, Package_TO_SOT_THT:TO-220-3_Vertical, symbol Regulator_Linear:LM1117-3.3
- added U2: AMS1117-3.3, Package_TO_SOT_SMD:SOT-223-3_TabPin2, symbol Regulator_Linear:AMS1117-3.3
Connections:
- net GND: now also U2.1 (GND)
- net LDO_in: now also U2.3 (VI)
- net LDO_out: now also U2.2 (VO)
Changed lines of the file:
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@@
 (kicad_sch (version 20211123) (generator eeschema)
   (paper "A4")
+  (junction (at 120.65 66.04) (diameter 0) (color 0 0 0 0)
+  )
   (junction (at 85.09 66.04) (diameter 0) (color 0 0 0 0)
-  )
-  (junction (at 120.65 66.04) (diameter 0) (color 0 0 0 0)
   )
   (wire (pts (xy 120.65 66.04) (xy 120.65 72.39))
@@
     (pin "1")
   )
-  (symbol (lib_id "Regulator_Linear:LM1117-3.3") (at 104.14 66.04 0) (unit 1)
-    (in_bom yes) (on_board yes) (fields_autoplaced)
-    (property "Reference" "U3" (id 0) (at 104.14 58.42 0))
-    (property "Value" "LM1117-3.3" (id 1) (at 104.14 60.96 0))
-    (property "Footprint" "Package_TO_SOT_THT:TO-220-3_Vertical" (id 2) (at 104.14 66.04 0)
-      (effects (font (size 1.27 1.27)) hide)
-    )
-    (property "Datasheet" "http://www.ti.com/lit/ds/symlink/lm1117.pdf" (id 3) (at 104.14 66.04 0)
-      (effects (font (size 1.27 1.27)) hide)
-    )
-    (pin "1")
-    (pin "2")
-    (pin "3")
-  )
   (symbol (lib_id "power:GND") (at 85.09 80.01 0) (unit 1)
     (in_bom yes) (on_board yes) (fields_autoplaced)
@@
     (pin "2")
   )
+  (symbol (lib_id "Regulator_Linear:AMS1117-3.3") (at 104.14 66.04 0) (unit 1)
+    (in_bom yes) (on_board yes) (fields_autoplaced)
+    (property "Reference" "U2" (id 0) (at 104.14 58.42 0))
+    (property "Value" "AMS1117-3.3" (id 1) (at 104.14 60.96 0))
+    (property "Footprint" "Package_TO_SOT_SMD:SOT-223-3_TabPin2" (id 2) (at 104.14 60.96 0)
+      (effects (font (size 1.27 1.27)) hide)
+    )
+    (property "Datasheet" "http://www.advanced-monolithic.com/pdf/ds1117.pdf" (id 3) (at 106.68 72.39 0)
+      (effects (font (size 1.27 1.27)) hide)
+    )
+    (pin "1")
+    (pin "2")
+    (pin "3")
+  )
 )

Commit message: Ruteo completo
Parts:
- renumbered C7 to C5, C8 to C6
Changed lines of the file:
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@@
   (symbol (lib_id "power:GND") (at 104.14 78.74 0) (unit 1)
     (in_bom yes) (on_board yes) (fields_autoplaced)
-    (property "Reference" "#PWR022" (id 0) (at 104.14 85.09 0)
+    (property "Reference" "#PWR030" (id 0) (at 104.14 85.09 0)
       (effects (font (size 1.27 1.27)) hide)
     )
@@
   (symbol (lib_id "Device:C_Polarized") (at 120.65 76.2 0) (unit 1)
     (in_bom yes) (on_board yes) (fields_autoplaced)
-    (property "Reference" "C8" (id 0) (at 124.46 74.0409 0)
+    (property "Reference" "C6" (id 0) (at 124.46 74.0409 0)
       (effects (font (size 1.27 1.27)) (justify left))
     )
@@
   (symbol (lib_id "power:GND") (at 120.65 80.01 0) (unit 1)
     (in_bom yes) (on_board yes) (fields_autoplaced)
-    (property "Reference" "#PWR023" (id 0) (at 120.65 86.36 0)
+    (property "Reference" "#PWR031" (id 0) (at 120.65 86.36 0)
       (effects (font (size 1.27 1.27)) hide)
     )
@@
   (symbol (lib_id "power:GND") (at 85.09 80.01 0) (unit 1)
     (in_bom yes) (on_board yes) (fields_autoplaced)
-    (property "Reference" "#PWR021" (id 0) (at 85.09 86.36 0)
+    (property "Reference" "#PWR029" (id 0) (at 85.09 86.36 0)
       (effects (font (size 1.27 1.27)) hide)
     )
@@
   (symbol (lib_id "Device:C_Polarized") (at 85.09 76.2 0) (unit 1)
     (in_bom yes) (on_board yes) (fields_autoplaced)
-    (property "Reference" "C7" (id 0) (at 88.9 74.0409 0)
+    (property "Reference" "C5" (id 0) (at 88.9 74.0409 0)
       (effects (font (size 1.27 1.27)) (justify left))
     )
