File: CircuitDesing/embebidos/Actuadores.kicad_sch (KiCad schematic)
At the start: 24 parts, among them Q2 IRF540N, Q3 IRF540N, Q4 IRF540N, Q5 IRF540N

Commit message: Jack, arreglos para disipacion
Changed lines of the file:
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@@
     (stroke (width 0) (type default) (color 0 0 0 0))
   )
-  (wire (pts (xy 236.22 105.41) (xy 236.22 107.95))
+  (wire (pts (xy 236.22 101.6) (xy 236.22 107.95))
     (stroke (width 0) (type default) (color 0 0 0 0))
   )
@@
     (effects (font (size 1.27 1.27)) (justify left bottom))
   )
-  (label "5v" (at 236.22 105.41 0)
-    (effects (font (size 1.27 1.27)) (justify left bottom))
-  )
+  (label "5v" (at 236.22 101.6 0)
+    (effects (font (size 1.27 1.27)) (justify left bottom))
+  )
