File: CircuitDesing/embebidos/embebidos.kicad_pcb (KiCad board)
At the start: 2 copper layers, 5 parts, among them U1 ESP32-WROOM-32

Commit message: Avance esquemático
Subcircuitos
Parts:
- added REF**: JST_XH_S3B-XH-A-1_1x03_P2.50mm_Horizontal, Connector_JST:JST_XH_S3B-XH-A-1_1x03_P2.50mm_Horizontal, F.Cu at (78.7, 129.5)
- added REF**: JST_XH_S3B-XH-A-1_1x03_P2.50mm_Horizontal, Connector_JST:JST_XH_S3B-XH-A-1_1x03_P2.50mm_Horizontal, F.Cu at (94.0, 129.5)
Changed lines of the file:
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@@
+    )
+  )
+  (footprint "Connector_JST:JST_XH_S3B-XH-A-1_1x03_P2.50mm_Horizontal" (layer "F.Cu")
+    (at 78.74 129.54)
+    (descr "JST XH series connector, S3B-XH-A-1 (http://www.jst-mfg.com/product/pdf/eng/eXH.pdf), generated with kicad-footprint-generator")
+    (tags "connector JST XH horizontal")
+    (attr through_hole)
+    (fp_text reference "REF**" (at 2.5 -5.1) (layer "F.SilkS")
+      (effects (font (size 1 1) (thickness 0.15)))
+    )
+    (fp_text value "JST_XH_S3B-XH-A-1_1x03_P2.50mm_Horizontal" (at 2.5 8.8) (layer "F.Fab")
+      (effects (font (size 1 1) (thickness 0.15)))
+    )
+    (fp_text user "${REFERENCE}" (at 2.5 1.85) (layer "F.Fab")
+      (effects (font (size 1 1) (thickness 0.15)))
+    )
+    (fp_line (start 6.14 -4.01) (end 6.14 0.49) (layer "F.SilkS") (width 0.12))
+    (fp_line (start 2.75 1.6) (end 2.25 1.6) (layer "F.SilkS") (width 0.12))
+    (fp_line (start -0.25 7.1) (end 0.25 7.1) (layer "F.SilkS") (width 0.12))
+    (fp_line (start 2.75 7.1) (end 2.75 1.6) (layer "F.SilkS") (width 0.12))
+    (fp_line (start 2.5 7.71) (end 7.56 7.71) (layer "F.SilkS") (width 0.12))
+    (fp_line (start 0.25 1.6) (end -0.25 1.6) (layer "F.SilkS") (width 0.12))
+    (fp_line (start -1.14 -4.01) (end -1.14 0.49) (layer "F.SilkS") (width 0.12))
+    (fp_line (start 2.25 7.1) (end 2.75 7.1) (layer "F.SilkS") (width 0.12))
+    (fp_line (start -2.56 -4.01) (end -1.14 -4.01) (layer "F.SilkS") (width 0.12))
+    (fp_line (start 7.56 -4.01) (end 6.14 -4.01) (layer "F.SilkS") (width 0.12))
+    (fp_line (start -0.25 1.6) (end -0.25 7.1) (layer "F.SilkS") (width 0.12))
+    (fp_line (start 5.25 7.1) (end 5.25 1.6) (layer "F.SilkS") (width 0.12))
+    (fp_line (start 4.75 1.6) (end 4.75 7.1) (layer "F.SilkS") (width 0.12))
+    (fp_line (start 0.3 -2.1) (end 0 -1.5) (layer "F.SilkS") (width 0.12))
+    (fp_line (start 5.25 1.6) (end 4.75 1.6) (layer "F.SilkS") (width 0.12))
+    (fp_line (start 7.56 7.71) (end 7.56 -4.01) (layer "F.SilkS") (width 0.12))
+    (fp_line (start 0.25 7.1) (end 0.25 1.6) (layer "F.SilkS") (width 0.12))
+    (fp_line (start 0 -1.5) (end -0.3 -2.1) (layer "F.SilkS") (width 0.12))
+    (fp_line (start 4.75 7.1) (end 5.25 7.1) (layer "F.SilkS") (width 0.12))
+    (fp_line (start 2.25 1.6) (end 2.25 7.1) (layer "F.SilkS") (width 0.12))
+    (fp_line (start -2.56 7.71) (end -2.56 -4.01) (layer "F.SilkS") (width 0.12))
+    (fp_line (start 2.5 7.71) (end -2.56 7.71) (layer "F.SilkS") (width 0.12))
+    (fp_line (start -0.3 -2.1) (end 0.3 -2.1) (layer "F.SilkS") (width 0.12))
+    (fp_line (start 7.95 8.1) (end 7.95 -4.4) (layer "F.CrtYd") (width 0.05))
+    (fp_line (start 7.95 -4.4) (end -2.95 -4.4) (layer "F.CrtYd") (width 0.05))
+    (fp_line (start -2.95 8.1) (end 7.95 8.1) (layer "F.CrtYd") (width 0.05))
+    (fp_line (start -2.95 -4.4) (end -2.95 8.1) (layer "F.CrtYd") (width 0.05))
+    (fp_line (start 7.45 7.6) (end 7.45 -3.9) (layer "F.Fab") (width 0.1))
+    (fp_line (start -2.45 7.6) (end -2.45 -3.9) (layer "F.Fab") (width 0.1))
+    (fp_line (start 6.25 -3.9) (end 6.25 0.6) (layer "F.Fab") (width 0.1))
+    (fp_line (start -0.625 0.6) (end 0 -0.4) (layer "F.Fab") (width 0.1))
+    (fp_line (start 2.5 7.6) (end -2.45 7.6) (layer "F.Fab") (width 0.1))
+    (fp_line (start 0 -0.4) (end 0.625 0.6) (layer "F.Fab") (width 0.1))
+    (fp_line (start -1.25 0.6) (end 2.5 0.6) (layer "F.Fab") (width 0.1))
+    (fp_line (start 2.5 7.6) (end 7.45 7.6) (layer "F.Fab") (width 0.1))
+    (fp_line (start -2.45 -3.9) (end -1.25 -3.9) (layer "F.Fab") (width 0.1))
+    (fp_line (start 7.45 -3.9) (end 6.25 -3.9) (layer "F.Fab") (width 0.1))
+    (fp_line (start -1.25 -3.9) (end -1.25 0.6) (layer "F.Fab") (width 0.1))
+    (fp_line (start 6.25 0.6) (end 2.5 0.6) (layer "F.Fab") (width 0.1))
+    (pad "1" thru_hole roundrect (at 0 0) (size 1.7 1.95) (drill 0.95) (layers *.Cu *.Mask) (roundrect_rratio 0.147059))
+    (pad "2" thru_hole oval (at 2.5 0) (size 1.7 1.95) (drill 0.95) (layers *.Cu *.Mask))
+    (pad "3" thru_hole oval (at 5 0) (size 1.7 1.95) (drill 0.95) (layers *.Cu *.Mask))
+    (model "${KICAD6_3DMODEL_DIR}/Connector_JST.3dshapes/JST_XH_S3B-XH-A-1_1x03_P2.50mm_Horizontal.wrl"
+      (offset (xyz 0 0 0))
+      (scale (xyz 1 1 1))
+      (rotate (xyz 0 0 0))
+    )
+  )
+  (footprint "Connector_JST:JST_XH_S3B-XH-A-1_1x03_P2.50mm_Horizontal" (layer "F.Cu")
+    (at 93.98 129.54)
+    (descr "JST XH series connector, S3B-XH-A-1 (http://www.jst-mfg.com/product/pdf/eng/eXH.pdf), generated with kicad-footprint-generator")
+    (tags "connector JST XH horizontal")
+    (attr through_hole)
+    (fp_text reference "REF**" (at 2.5 -5.1) (layer "F.SilkS")
+      (effects (font (size 1 1) (thickness 0.15)))
+    )
+    (fp_text value "JST_XH_S3B-XH-A-1_1x03_P2.50mm_Horizontal" (at 2.5 8.8) (layer "F.Fab")
+      (effects (font (size 1 1) (thickness 0.15)))
+    )
+    (fp_text user "${REFERENCE}" (at 2.5 1.85) (layer "F.Fab")
+      (effects (font (size 1 1) (thickness 0.15)))
+    )
+    (fp_line (start -2.56 7.71) (end -2.56 -4.01) (layer "F.SilkS") (width 0.12))
+    (fp_line (start 0.25 1.6) (end -0.25 1.6) (layer "F.SilkS") (width 0.12))
+    (fp_line (start 2.5 7.71) (end 7.56 7.71) (layer "F.SilkS") (width 0.12))
+    (fp_line (start -0.25 1.6) (end -0.25 7.1) (layer "F.SilkS") (width 0.12))
+    (fp_line (start 2.75 1.6) (end 2.25 1.6) (layer "F.SilkS") (width 0.12))
+    (fp_line (start 7.56 7.71) (end 7.56 -4.01) (layer "F.SilkS") (width 0.12))
+    (fp_line (start 6.14 -4.01) (end 6.14 0.49) (layer "F.SilkS") (width 0.12))
+    (fp_line (start 2.5 7.71) (end -2.56 7.71) (layer "F.SilkS") (width 0.12))
+    (fp_line (start -0.3 -2.1) (end 0.3 -2.1) (layer "F.SilkS") (width 0.12))
+    (fp_line (start 5.25 7.1) (end 5.25 1.6) (layer "F.SilkS") (width 0.12))
+    (fp_line (start 7.56 -4.01) (end 6.14 -4.01) (layer "F.SilkS") (width 0.12))
+    (fp_line (start -2.56 -4.01) (end -1.14 -4.01) (layer "F.SilkS") (width 0.12))
+    (fp_line (start 0.3 -2.1) (end 0 -1.5) (layer "F.SilkS") (width 0.12))
+    (fp_line (start 4.75 7.1) (end 5.25 7.1) (layer "F.SilkS") (width 0.12))
+    (fp_line (start 0 -1.5) (end -0.3 -2.1) (layer "F.SilkS") (width 0.12))
+    (fp_line (start 0.25 7.1) (end 0.25 1.6) (layer "F.SilkS") (width 0.12))
+    (fp_line (start 5.25 1.6) (end 4.75 1.6) (layer "F.SilkS") (width 0.12))
+    (fp_line (start -0.25 7.1) (end 0.25 7.1) (layer "F.SilkS") (width 0.12))
+    (fp_line (start 2.25 7.1) (end 2.75 7.1) (layer "F.SilkS") (width 0.12))
+    (fp_line (start 2.75 7.1) (end 2.75 1.6) (layer "F.SilkS") (width 0.12))
+    (fp_line (start 2.25 1.6) (end 2.25 7.1) (layer "F.SilkS") (width 0.12))
+    (fp_line (start 4.75 1.6) (end 4.75 7.1) (layer "F.SilkS") (width 0.12))
+    (fp_line (start -1.14 -4.01) (end -1.14 0.49) (layer "F.SilkS") (width 0.12))
+    (fp_line (start -2.95 8.1) (end 7.95 8.1) (layer "F.CrtYd") (width 0.05))
+    (fp_line (start 7.95 -4.4) (end -2.95 -4.4) (layer "F.CrtYd") (width 0.05))
+    (fp_line (start 7.95 8.1) (end 7.95 -4.4) (layer "F.CrtYd") (width 0.05))
+    (fp_line (start -2.95 -4.4) (end -2.95 8.1) (layer "F.CrtYd") (width 0.05))
+    (fp_line (start -2.45 7.6) (end -2.45 -3.9) (layer "F.Fab") (width 0.1))
+    (fp_line (start -2.45 -3.9) (end -1.25 -3.9) (layer "F.Fab") (width 0.1))
+    (fp_line (start 6.25 0.6) (end 2.5 0.6) (layer "F.Fab") (width 0.1))
+    (fp_line (start 2.5 7.6) (end -2.45 7.6) (layer "F.Fab") (width 0.1))
+    (fp_line (start 7.45 7.6) (end 7.45 -3.9) (layer "F.Fab") (width 0.1))
+    (fp_line (start 2.5 7.6) (end 7.45 7.6) (layer "F.Fab") (width 0.1))
+    (fp_line (start -0.625 0.6) (end 0 -0.4) (layer "F.Fab") (width 0.1))
+    (fp_line (start -1.25 -3.9) (end -1.25 0.6) (layer "F.Fab") (width 0.1))
+    (fp_line (start 7.45 -3.9) (end 6.25 -3.9) (layer "F.Fab") (width 0.1))
+    (fp_line (start 6.25 -3.9) (end 6.25 0.6) (layer "F.Fab") (width 0.1))
+    (fp_line (start -1.25 0.6) (end 2.5 0.6) (layer "F.Fab") (width 0.1))
+    (fp_line (start 0 -0.4) (end 0.625 0.6) (layer "F.Fab") (width 0.1))
+    (pad "1" thru_hole roundrect (at 0 0) (size 1.7 1.95) (drill 0.95) (layers *.Cu *.Mask) (roundrect_rratio 0.147059))
+    (pad "2" thru_hole oval (at 2.5 0) (size 1.7 1.95) (drill 0.95) (layers *.Cu *.Mask))
+    (pad "3" thru_hole oval (at 5 0) (size 1.7 1.95) (drill 0.95) (layers *.Cu *.Mask))
+    (model "${KICAD6_3DMODEL_DIR}/Connector_JST.3dshapes/JST_XH_S3B-XH-A-1_1x03_P2.50mm_Horizontal.wrl"
+      (offset (xyz 0 0 0))
+      (scale (xyz 1 1 1))
+      (rotate (xyz 0 0 0))
     )
   )

Commit message: Huellas parciales
Parts:
- added 10k1: R, Resistor_SMD:R_0603_1608Metric_Pad0.98x0.95mm_HandSolder, F.Cu at (124.4, 124.0)
- added 10k2: R, Resistor_SMD:R_0603_1608Metric_Pad0.98x0.95mm_HandSolder, F.Cu at (114.3, 106.3)
- added 7k1: R, Resistor_SMD:R_0603_1608Metric_Pad0.98x0.95mm_HandSolder, F.Cu at (124.4, 101.2)
- added Bomba1: Conn_01x02, Connector_JST:JST_EH_B2B-EH-A_1x02_P2.50mm_Vertical, F.Cu at (170.2, 129.5)
- added C4: 470u, Capacitor_SMD:C_0603_1608Metric_Pad1.08x0.95mm_HandSolder, F.Cu at (136.0, 123.2)
- added C5: 100u, Capacitor_SMD:C_0603_1608Metric_Pad1.08x0.95mm_HandSolder, F.Cu at (126.1, 114.3)
- added C6: 1000u, Capacitor_SMD:C_0603_1608Metric_Pad1.08x0.95mm_HandSolder, F.Cu at (126.1, 116.8)
- added C7: 10u, Capacitor_SMD:C_0603_1608Metric_Pad1.08x0.95mm_HandSolder, F.Cu at (111.2, 126.6)
- added C8: 100u, Capacitor_SMD:C_0603_1608Metric_Pad1.08x0.95mm_HandSolder, F.Cu at (111.2, 124.0)
- added D1: 1N5822, Diode_THT:D_DO-201AD_P15.24mm_Horizontal, F.Cu at (175.3, 86.4)
- added D11: 1N4004, Diode_THT:D_DO-41_SOD81_P10.16mm_Horizontal, F.Cu at (174.8, 110.7)
- added D2: 1N5822, Diode_THT:D_DO-201AD_P15.24mm_Horizontal, F.Cu at (175.3, 93.1)
- added D3: 1N5822, Diode_THT:D_DO-201AD_P15.24mm_Horizontal, F.Cu at (195.2, 79.6)
- added D4: 1N5822, Diode_THT:D_DO-201AD_P15.24mm_Horizontal, F.Cu at (175.3, 79.6)
- added D5: 1N5822, Diode_THT:D_DO-201AD_P15.24mm_Horizontal, F.Cu at (222.8, 79.6)
- added D7: 1N4004, Diode_THT:D_DO-41_SOD81_P10.16mm_Horizontal, F.Cu at (188.7, 106.4)
- added D9: 1N4004, Diode_THT:D_DO-41_SOD81_P10.16mm_Horizontal, F.Cu at (174.8, 106.4)
- added Q1: IRF540N, Package_TO_SOT_THT:TO-220-3_Vertical, F.Cu at (176.1, 116.7)
- added Q2: IRF540N, Package_TO_SOT_THT:TO-220-3_Vertical, F.Cu at (190.0, 112.5)
- added Q3: IRF540N, Package_TO_SOT_THT:TO-220-3_Vertical, F.Cu at (187.7, 118.5)
- added U2: LM2576S-5, Package_TO_SOT_SMD:TO-263-5_TabPin3, F.Cu at (229.3, 89.2)
- moved REF** 63.6 mm to (142.2, 132.1)
- moved REF** 63.6 mm to (157.5, 132.1)
- moved U1 22.9 mm to (134.6, 78.9)
- moved C2 18.2 mm to (134.7, 100.9)
- moved R1 18.2 mm to (134.7, 103.5)
Connections:
- net +3.3V renamed /3.3v
- U1 pad 10: unconnected-(U1-Pad10) -> /Esp32Schematic/IO25
- U1 pad 11: unconnected-(U1-Pad11) -> /Esp32Schematic/IO26
- U1 pad 12: unconnected-(U1-Pad12) -> /Esp32Schematic/IO27
- U1 pad 13: unconnected-(U1-Pad13) -> /Esp32Schematic/IO14
- U1 pad 14: unconnected-(U1-Pad14) -> /Esp32Schematic/IO12
- U1 pad 16: unconnected-(U1-Pad16) -> /Esp32Schematic/IO13
- U1 pad 23: unconnected-(U1-Pad23) -> /HC-SR04Echo
- U1 pad 24: unconnected-(U1-Pad24) -> /HC-SR04Trig
- U1 pad 25: unconnected-(U1-Pad25) -> /Esp32Schematic/BOOT
- U1 pad 26: unconnected-(U1-Pad26) -> /Esp32Schematic/IO4
- U1 pad 27: unconnected-(U1-Pad27) -> /dht11_1d
- U1 pad 28: unconnected-(U1-Pad28) -> /dht11_2d
- U1 pad 29: unconnected-(U1-Pad29) -> /Esp32Schematic/IO5
- U1 pad 30: unconnected-(U1-Pad30) -> /c_vent1
- U1 pad 31: unconnected-(U1-Pad31) -> /c_vent2
- U1 pad 33: unconnected-(U1-Pad33) -> /c_bomba
- U1 pad 34: unconnected-(U1-Pad34) -> /Esp32Schematic/RXD0/IO3
- U1 pad 35: unconnected-(U1-Pad35) -> /Esp32Schematic/TXD0/IO1
- U1 pad 36: unconnected-(U1-Pad36) -> /Esp32Schematic/IO22
- U1 pad 37: unconnected-(U1-Pad37) -> /Esp32Schematic/IO23
- U1 pad 6: unconnected-(U1-Pad6) -> /lm393_d
- U1 pad 7: unconnected-(U1-Pad7) -> /se093_d
- U1 pad 8: unconnected-(U1-Pad8) -> /Esp32Schematic/IO32
- U1 pad 9: unconnected-(U1-Pad9) -> /Esp32Schematic/IO33
Routing:
- net /3.3v: track 108.0 -> 0.07 mm
- net GND: track 68.3 -> 2.62 mm

Commit message: 15 footprints faltantes
Parts:
- added HC-SR4: Conn_01x04, Connector_JST:JST_EH_B4B-EH-A_1x04_P2.50mm_Vertical, F.Cu at (180.3, 129.5)
- added R2: 1k, Resistor_SMD:R_0603_1608Metric_Pad0.98x0.95mm_HandSolder, F.Cu at (160.0, 106.7)
- added R3: 1k, Resistor_SMD:R_0603_1608Metric_Pad0.98x0.95mm_HandSolder, F.Cu at (160.0, 104.2)
- added R4: 1k, Resistor_SMD:R_0603_1608Metric_Pad0.98x0.95mm_HandSolder, F.Cu at (164.4, 104.2)
- added R5: 1k, Resistor_SMD:R_0603_1608Metric_Pad0.98x0.95mm_HandSolder, F.Cu at (164.4, 106.7)
- added R6: 1k, Resistor_SMD:R_0603_1608Metric_Pad0.98x0.95mm_HandSolder, F.Cu at (160.0, 109.2)
- added R7: 1k, Resistor_SMD:R_0603_1608Metric_Pad0.98x0.95mm_HandSolder, F.Cu at (168.7, 104.2)
- moved Q2 14.2 mm to (200.7, 121.9)

Commit message: Todas las huellas
Parts:
- added D10: LED, LED_SMD:LED_0603_1608Metric_Pad1.05x0.95mm_HandSolder, F.Cu at (185.3, 69.3)
- added D6: LED, LED_SMD:LED_0603_1608Metric_Pad1.05x0.95mm_HandSolder, F.Cu at (190.5, 63.5)
- added D8: LED, LED_SMD:LED_0603_1608Metric_Pad1.05x0.95mm_HandSolder, F.Cu at (180.9, 69.3)
- added DHT11_1: Conn_01x03, Connector_JST:JST_EH_B3B-EH-A_1x03_P2.50mm_Vertical, F.Cu at (81.3, 88.9)
- added DHT11_2: Conn_01x03, Connector_JST:JST_EH_B3B-EH-A_1x03_P2.50mm_Vertical, F.Cu at (93.3, 83.0)
- added J1: Conn_01x02, Connector_JST:JST_EH_B2B-EH-A_1x02_P2.50mm_Vertical, F.Cu at (97.5, 101.7)
- added L1: 100u, Inductor_SMD:L_0603_1608Metric_Pad1.05x0.95mm_HandSolder, F.Cu at (110.8, 90.7)
- added SE93: Conn_01x03, Connector_JST:JST_EH_B3B-EH-A_1x03_P2.50mm_Vertical, F.Cu at (81.3, 83.0)
- added SW1: SW_Push, Button_Switch_SMD:SW_SPST_EVQP0, F.Cu at (167.2, 66.0)
- added SW2: SW_Push, Button_Switch_SMD:SW_SPST_EVQP0, F.Cu at (157.1, 66.0)
- added U3: LM1117-3.3, Package_TO_SOT_THT:TO-220-3_Vertical, F.Cu at (81.0, 103.0)
- added Vent1: Conn_01x02, Connector_JST:JST_EH_B2B-EH-A_1x02_P2.50mm_Vertical, F.Cu at (112.2, 83.0)
- added Vent2: Conn_01x02, Connector_JST:JST_EH_B2B-EH-A_1x02_P2.50mm_Vertical, F.Cu at (182.3, 64.8)

Commit message: Actualizacion huellas
Huellas+Programador
Parts:
- removed C5: 100u, Capacitor_SMD:C_0603_1608Metric_Pad1.08x0.95mm_HandSolder
- removed C6: 1000u, Capacitor_SMD:C_0603_1608Metric_Pad1.08x0.95mm_HandSolder
- removed D1, D2, D3, D4, D5: 1N5822, Diode_THT:D_DO-201AD_P15.24mm_Horizontal
- removed L1: 100u, Inductor_SMD:L_0603_1608Metric_Pad1.05x0.95mm_HandSolder
- removed REF** (x2): JST_XH_S3B-XH-A-1_1x03_P2.50mm_Horizontal, Connector_JST:JST_XH_S3B-XH-A-1_1x03_P2.50mm_Horizontal
- added 10k3: R, Resistor_SMD:R_0603_1608Metric_Pad0.98x0.95mm_HandSolder, F.Cu at (210.8, 108.2)
- added 10k4: R, Resistor_SMD:R_0603_1608Metric_Pad0.98x0.95mm_HandSolder, F.Cu at (220.3, 102.4)
- added J2: USB_B_Micro, Connector_USB:USB_Micro-B_Amphenol_10118194_Horizontal, F.Cu at (150.5, 99.6)
- added J_I2C1: Conn_01x05_Male, Connector_PinSocket_2.54mm:PinSocket_1x05_P2.54mm_Horizontal, F.Cu at (131.7, 98.8)
- added J_prog1: Conn_01x06_Male, Connector_PinHeader_2.54mm:PinHeader_1x06_P2.54mm_Horizontal, F.Cu at (109.5, 98.8)
- added L_p1: LED, LED_SMD:LED_0805_2012Metric_Pad1.15x1.40mm_HandSolder, F.Cu at (123.0, 112.8)
- added Q4: 2N2219, Package_TO_SOT_THT:TO-39-3, F.Cu at (211.5, 95.7)
- added R8: 10k, Resistor_SMD:R_0603_1608Metric_Pad0.98x0.95mm_HandSolder, F.Cu at (113.8, 89.4)
- added RCL1: 10k, Resistor_SMD:R_0805_2012Metric_Pad1.20x1.40mm_HandSolder, F.Cu at (127.8, 112.7)
- added RDA1: 10k, Resistor_SMD:R_0805_2012Metric_Pad1.20x1.40mm_HandSolder, F.Cu at (136.3, 100.9)
- added R_p1: 47, Resistor_SMD:R_0805_2012Metric_Pad1.20x1.40mm_HandSolder, F.Cu at (136.3, 98.0)
- added U4: LM741, Package_DFN_QFN:DFN-8-1EP_2x2mm_P0.5mm_EP1.05x1.75mm, F.Cu at (221.5, 97.0)
- C1: value 10uF -> 1uF
- C3: value 1uF -> 10uF
- C4: value 470u -> 1uF
- SW1, SW2: footprint Button_Switch_SMD:SW_SPST_EVQP0 -> Button_Switch_SMD:SW_Push_1P1T_NO_6x6mm_H9.5mm
- U2: value LM2576S-5 -> AMS1117-3.3; footprint Package_TO_SOT_SMD:TO-263-5_TabPin3 -> Package_TO_SOT_SMD:SOT-223-3_TabPin2
- U3: value LM1117-3.3 -> LM4250; footprint Package_TO_SOT_THT:TO-220-3_Vertical -> Package_DFN_QFN:DFN-8-1EP_2x2mm_P0.5mm_EP1.05x1.75mm
- moved U3 145.1 mm to (225.8, 94.5)
- moved DHT11_1 142.7 mm to (220.6, 58.3)
- moved SE93 126.2 mm to (206.1, 64.1)
- moved J1 114.6 mm to (212.1, 103.8)
- moved DHT11_2 113.5 mm to (206.1, 70.0)
- moved 10k2 108.4 mm to (221.7, 91.4)
- moved 7k1 102.1 mm to (226.1, 91.4)
- moved 10k1 101.8 mm to (221.7, 94.0)
- moved C7 85.4 mm to (189.1, 91.4)
- moved HC-SR4 75.8 mm to (206.1, 58.3)
- moved C8 72.3 mm to (179.2, 99.7)
- moved Vent1 69.0 mm to (180.6, 74.3)
- moved Q2 60.8 mm to (182.7, 63.8)
- moved Bomba1 50.9 mm to (169.0, 78.7)
- moved D11 49.2 mm to (167.4, 62.0)
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Connections:
- 10k1 pad 1: /5v -> 5v
- Bomba1 pad 2: /5v -> 5v
- C1 pad 1: /3.3v -> GND
- C1 pad 2: GND -> Net-(C1-Pad2)
- C2 pad 1: /3.3v -> 3.3v
- C3 pad 1: GND -> 3.3v
- C3 pad 2: Net-(C3-Pad2) -> GND
- C4 pad 1: /Potencia/out_rect -> /Esp32Schematic/BOOT
- D11 pad 1: /5v -> 5v
- D7 pad 1: /5v -> 5v
- D9 pad 1: /5v -> 5v
- DHT11_1 pad 1: /5v -> /Sensores/3.3v
- DHT11_2 pad 1: /5v -> /Sensores/3.3v
- HC-SR4 pad 1: /5v -> 5v
- J1 pad 1: /5v -> 5v
- R1 pad 1: /3.3v -> 3.3v
- R1 pad 2: Net-(C3-Pad2) -> Net-(C1-Pad2)
- SE93 pad 1: /5v -> /Sensores/3.3v
- SW1 pad 2: Net-(C3-Pad2) -> Net-(C1-Pad2)
- U1 pad 13: /Esp32Schematic/IO14 -> /HC-SR04Trig
- U1 pad 16: /Esp32Schematic/IO13 -> /c_bomba
- U1 pad 2: /3.3v -> 3.3v
- U1 pad 24: /HC-SR04Trig -> /Esp32Schematic/IO2
- U1 pad 3: Net-(C3-Pad2) -> Net-(C1-Pad2)
- U1 pad 33: /c_bomba -> SDA
- U1 pad 34: /Esp32Schematic/RXD0/IO3 -> /Prog_Tx
- U1 pad 35: /Esp32Schematic/TXD0/IO1 -> /Prog_Rx
- U1 pad 36: /Esp32Schematic/IO22 -> SCL
- U1 pad 5: unconnected-(U1-Pad5) -> /LedU1
- U2 pad 1: /Potencia/out_rect -> GND
- U2 pad 2: Net-(D5-Pad1) -> /Potencia/LDO/LDO_out
- U2 pad 3: GND -> /Potencia/LDO/LDO_in
- U3 pad 1: GND -> unconnected-(U3-Pad1)
- U3 pad 2: /Potencia/LDO/LDO_out -> unconnected-(U3-Pad2)
- U3 pad 3: /Potencia/LDO/LDO_in -> unconnected-(U3-Pad3)
- Vent1 pad 2: /5v -> 5v
- Vent2 pad 2: /5v -> 5v
Routing:
- net GND: track 2.62 -> 0.00 mm
