File: CircuitDesing/embebidos/embebidos.kicad_pcb (KiCad board)
At the start: 2 copper layers, 50 parts, among them J1 Conn_01x02, J2 USB_B_Micro, Q1 IRF540N, Q2 IRF540N, Q3 IRF540N, Q4 2N2219, SW1 SW_Push, SW2 SW_Push, U1 ESP32-WROOM-32, U2 AMS1117-3.3, U3 LM4250, U4 LM741

Commit message: Ruteo completo
Parts:
- removed J_prog1: Conn_01x06_Male, Connector_PinHeader_2.54mm:PinHeader_1x06_P2.54mm_Horizontal
- removed SW1, SW2: SW_Push, Button_Switch_SMD:SW_Push_1P1T_NO_6x6mm_H9.5mm
- removed U4: LM741, Package_DFN_QFN:DFN-8-1EP_2x2mm_P0.5mm_EP1.05x1.75mm
- added BOOT1: SW_Push, Button_Switch_SMD:SW_Push_1P1T_NO_6x6mm_H9.5mm, F.Cu at (136.1, 51.8)
- added Botones_M1: Conn_01x03, Connector_JST:JST_EH_B3B-EH-A_1x03_P2.50mm_Vertical, F.Cu at (59.7, 76.7)
- added Buzzer1: Conn_01x02, Connector_JST:JST_EH_B2B-EH-A_1x02_P2.50mm_Vertical, F.Cu at (59.7, 116.6)
- added D5: LED, LED_SMD:LED_0603_1608Metric_Pad1.05x0.95mm_HandSolder, F.Cu at (87.4, 93.7)
- added D7: 1N4004, Diode_THT:D_DO-41_SOD81_P10.16mm_Horizontal, F.Cu at (96.8, 131.3)
- added EN1: SW_Push, Button_Switch_SMD:SW_Push_1P1T_NO_6x6mm_H9.5mm, F.Cu at (81.8, 54.9)
- added Humi1: Conn_01x02, Connector_JST:JST_EH_B2B-EH-A_1x02_P2.50mm_Vertical, F.Cu at (93.7, 136.1)
- added J1: Conn_01x03_Male, Connector_PinHeader_2.54mm:PinHeader_1x03_P2.54mm_Vertical, F.Cu at (150.4, 63.8)
- added LedRojo1: Conn_01x02, Connector_JST:JST_EH_B2B-EH-A_1x02_P2.50mm_Vertical, F.Cu at (59.7, 107.2)
- added LedVerde1: Conn_01x02, Connector_JST:JST_EH_B2B-EH-A_1x02_P2.50mm_Vertical, F.Cu at (59.7, 125.5)
- added Pantalla-I2C1: Conn_01x04, Connector_JST:JST_EH_B4B-EH-A_1x04_P2.50mm_Vertical, F.Cu at (148.5, 99.5)
- added Q1: BSS138, Package_TO_SOT_SMD:SOT-23, F.Cu at (67.1, 110.2)
- added Q10: BSS138, Package_TO_SOT_SMD:SOT-23, F.Cu at (68.3, 137.2)
- added Q11: BSS138, Package_TO_SOT_SMD:SOT-23, F.Cu at (132.1, 67.6)
- added Q12: BSS138, Package_TO_SOT_SMD:SOT-23, F.Cu at (80.0, 138.4)
- added Q13: BSS138, Package_TO_SOT_SMD:SOT-23, F.Cu at (96.0, 79.0)
- added Q14: BSS138, Package_TO_SOT_SMD:SOT-23, F.Cu at (62.2, 138.9)
- added Q15: BSS138, Package_TO_SOT_SMD:SOT-23, F.Cu at (86.6, 73.9)
- added Q16: BSS138, Package_TO_SOT_SMD:SOT-23, F.Cu at (114.3, 79.0)
- added Q6: BSS138, Package_TO_SOT_SMD:SOT-23, F.Cu at (104.6, 79.0)
- added Q7: BSS138, Package_TO_SOT_SMD:SOT-23, F.Cu at (74.4, 138.4)
- added Q8: MMBT3904, Package_TO_SOT_SMD:SOT-23, F.Cu at (83.1, 66.3)
- added Q9: BSS138, Package_TO_SOT_SMD:SOT-23, F.Cu at (126.0, 67.6)
- added R11: 10k, Resistor_SMD:R_0603_1608Metric_Pad0.98x0.95mm_HandSolder, F.Cu at (108.0, 79.0)
- added R12: 10k, Resistor_SMD:R_0603_1608Metric_Pad0.98x0.95mm_HandSolder, F.Cu at (99.6, 99.2)
- added R13: 10k, Resistor_SMD:R_0603_1608Metric_Pad0.98x0.95mm_HandSolder, F.Cu at (74.7, 135.6)
- added R14: 10k, Resistor_SMD:R_0603_1608Metric_Pad0.98x0.95mm_HandSolder, F.Cu at (74.7, 134.1)
- added R15: 10k, Resistor_SMD:R_0603_1608Metric_Pad0.98x0.95mm_HandSolder, F.Cu at (126.0, 64.3)
- added R16: 10k, Resistor_SMD:R_0603_1608Metric_Pad0.98x0.95mm_HandSolder, F.Cu at (116.8, 93.0)
- added R17: 10k, Resistor_SMD:R_0603_1608Metric_Pad0.98x0.95mm_HandSolder, F.Cu at (68.2, 133.1)
- added R18: 10k, Resistor_SMD:R_0603_1608Metric_Pad0.98x0.95mm_HandSolder, F.Cu at (68.3, 134.6)
- added R19: 10k, Resistor_SMD:R_0603_1608Metric_Pad0.98x0.95mm_HandSolder, F.Cu at (132.1, 64.3)
- added R20: 10k, Resistor_SMD:R_0603_1608Metric_Pad0.98x0.95mm_HandSolder, F.Cu at (137.2, 69.1)
- added R21: 10k, Resistor_SMD:R_0603_1608Metric_Pad0.98x0.95mm_HandSolder, F.Cu at (80.0, 135.9)
- added R22: 10k, Resistor_SMD:R_0603_1608Metric_Pad0.98x0.95mm_HandSolder, F.Cu at (80.0, 134.4)
- added R23: 10k, Resistor_SMD:R_0603_1608Metric_Pad0.98x0.95mm_HandSolder, F.Cu at (99.3, 79.0)
- added R24: 10k, Resistor_SMD:R_0603_1608Metric_Pad0.98x0.95mm_HandSolder, F.Cu at (94.5, 74.9)
- added R25: 10k, Resistor_SMD:R_0603_1608Metric_Pad0.98x0.95mm_HandSolder, F.Cu at (62.3, 136.4)
- added R26: 10k, Resistor_SMD:R_0603_1608Metric_Pad0.98x0.95mm_HandSolder, F.Cu at (62.2, 134.9)
- added R27: 10k, Resistor_SMD:R_0603_1608Metric_Pad0.98x0.95mm_HandSolder, F.Cu at (89.9, 73.9)
- added R28: 10k, Resistor_SMD:R_0603_1608Metric_Pad0.98x0.95mm_HandSolder, F.Cu at (84.6, 77.7)
- added R29: 10k, Resistor_SMD:R_0603_1608Metric_Pad0.98x0.95mm_HandSolder, F.Cu at (117.6, 79.0)
- added R30: 10k, Resistor_SMD:R_0603_1608Metric_Pad0.98x0.95mm_HandSolder, F.Cu at (113.3, 84.6)
- added R7: 1k, Resistor_SMD:R_0603_1608Metric_Pad0.98x0.95mm_HandSolder, F.Cu at (96.3, 93.7)
- added R9: 1k, Resistor_SMD:R_0603_1608Metric_Pad0.98x0.95mm_HandSolder, F.Cu at (87.4, 90.2)
- added RCL1: 10k, Resistor_SMD:R_0805_2012Metric_Pad1.20x1.40mm_HandSolder, F.Cu at (135.1, 83.6)
- added RDA1: 10k, Resistor_SMD:R_0805_2012Metric_Pad1.20x1.40mm_HandSolder, F.Cu at (135.4, 75.4)
- added R_p2: 47, Resistor_SMD:R_0805_2012Metric_Pad1.20x1.40mm_HandSolder, F.Cu at (78.7, 114.0)
- added R_p3: 1k, Resistor_SMD:R_0805_2012Metric_Pad1.20x1.40mm_HandSolder, F.Cu at (67.8, 105.4)
- added Rb1: 1k, Resistor_SMD:R_0603_1608Metric_Pad0.98x0.95mm_HandSolder, F.Cu at (67.3, 114.3)
- Q4: value 2N2219 -> IRF540N; footprint Package_TO_SOT_THT:TO-39-3 -> Package_TO_SOT_THT:TO-220-3_Vertical
- U3: footprint Package_DFN_QFN:DFN-8-1EP_2x2mm_P0.5mm_EP1.05x1.75mm -> Package_DIP:DIP-8_W7.62mm_SMDSocket_SmallPads
- moved 7k1 155.1 mm to (71.1, 84.8), turned to 180 degrees
- moved 10k1 154.6 mm to (68.1, 76.7)
- moved 10k2 154.1 mm to (68.1, 79.5), turned to 180 degrees
- moved J3 152.5 mm to (59.7, 97.8), turned to -90 degrees
- moved U3 150.6 mm to (76.2, 77.2)
- moved SE1 146.1 mm to (59.9, 64.3), turned to -90 degrees
- moved 10k4 143.1 mm to (83.1, 62.0), turned to 90 degrees
- moved 10k3 139.7 mm to (77.2, 67.3)
- moved C5 130.9 mm to (66.5, 45.2)
- moved HC-SR1 129.2 mm to (102.9, 136.1)
- moved U2 123.1 mm to (66.8, 50.8), turned to -90 degrees
- moved Q4 121.1 mm to (90.7, 87.4), turned to -90 degrees
- moved Bomba1 109.8 mm to (59.7, 88.6), turned to -90 degrees
- moved D2 107.0 mm to (92.1, 96.3)
- moved J2 106.0 mm to (56.3, 50.8), turned to -90 degrees
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- renumbered C7 to C5, C8 to C6, D6 to D1, D10 to D2, D7 to D3, D11 to D4, D8 to D6, D9 to D8, HC-SR4 to HC-SR1, J1 to J3, Q1 to Q2, Q2 to Q5, R5 to R10, R8 to R2, R2 to R3, R6 to R4, R3 to R5, R7 to R6, R4 to R8, RCL1 to RCL2, RDA1 to RDA2, SE93 to SE1
Connections:
- 10k3 pad 1: Net-(U4-Pad6) -> Net-(10k3-Pad1)
- C5 pad 1: /Potencia/LDO/LDO_in -> 5v
- C6 pad 1: /Potencia/LDO/LDO_out -> 3.3v
- DHT11_1 pad 1: /Sensores/3.3v -> 3.3v
- DHT11_2 pad 1: /Sensores/3.3v -> 3.3v
- HC-SR1 pad 2: /HC-SR04Trig -> /Sensores/Conversor_NLog5/HV1
- HC-SR1 pad 3: /HC-SR04Echo -> /Sensores/Conversor_NLog5/HV2
- J2 pad 1: /Potencia/IN_5v -> 5v
- Q2 pad 1: /c_vent1 -> /Actuadores/Conversor_NLog1/HV1
- Q3 pad 1: /c_bomba -> /Actuadores/Conversor_NLog3/HV1
- Q4 pad 1: /lm393_d -> /Actuadores/Conversor_NLog4/HV1
- Q4 pad 2: Net-(10k3-Pad2) -> Net-(D7-Pad2)
- Q4 pad 3: /Sensores/3.3v -> GND
- Q5 pad 1: /c_vent2 -> /Actuadores/Conversor_NLog2/HV1
- R10 pad 1: /c_vent2 -> /Actuadores/Conversor_NLog2/HV1
- R3 pad 1: /c_vent1 -> /Actuadores/Conversor_NLog1/HV1
- R4 pad 1: /c_bomba -> /Actuadores/Conversor_NLog3/HV1
- R5 pad 1: /c_vent1 -> /Actuadores/Conversor_NLog1/HV1
- R6 pad 1: /c_bomba -> /Actuadores/Conversor_NLog3/HV1
- R8 pad 1: /c_vent2 -> /Actuadores/Conversor_NLog2/HV1
- SE1 pad 1: /Sensores/3.3v -> 3.3v
- U1 pad 10: /Esp32Schematic/IO25 -> /Led_Verde
- U1 pad 14: /Esp32Schematic/IO12 -> /c_hum
- U1 pad 37: /Esp32Schematic/IO23 -> /Buzzer
- U1 pad 6: /lm393_d -> /Botones
- U1 pad 9: /Esp32Schematic/IO33 -> /lm393_d
- U2 pad 2: /Potencia/LDO/LDO_out -> 3.3v
- U2 pad 3: /Potencia/LDO/LDO_in -> 5v
- U3 pad 1: unconnected-(U3-Pad1) -> Net-(10k3-Pad1)
- U3 pad 2: unconnected-(U3-Pad2) -> Net-(10k1-Pad2)
- U3 pad 3: unconnected-(U3-Pad3) -> Net-(7k1-Pad1)
- U3 pad 4: unconnected-(U3-Pad4) -> GND
- U3 pad 8: unconnected-(U3-Pad8) -> 5v
Routing:
- net GND: track 0.00 -> 531.4 mm, vias 0 -> 4
- net 3.3v: track 0.00 -> 456.4 mm, vias 0 -> 11
- net 5v: track 0.00 -> 363.2 mm, vias 0 -> 17
- net /Buzzer: track 0.00 -> 96.0 mm, vias 0 -> 4
- net /Sensores/Conversor_NLog5/HV1: track 0.00 -> 76.1 mm
- net /dht11_1d: track 0.00 -> 71.3 mm
- net /Sensores/Conversor_NLog5/HV2: track 0.00 -> 66.2 mm
- net SCL: track 0.00 -> 66.1 mm, vias 0 -> 2
- net /dht11_2d: track 0.00 -> 60.7 mm
- net /Led_Verde: track 0.00 -> 57.7 mm, vias 0 -> 4
- net SDA: track 0.00 -> 56.4 mm, vias 0 -> 2
- net Net-(Bomba1-Pad1): track 0.00 -> 56.3 mm
- net /Actuadores/Conversor_NLog2/HV1: track 0.00 -> 52.8 mm, vias 0 -> 1
- net Net-(D7-Pad2): track 0.00 -> 52.2 mm
- net /Esp32Schematic/BOOT: track 0.00 -> 51.2 mm, vias 0 -> 2
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
Commit message: Ruteo plano a tierra
Parts:
- removed Q10, Q12, Q14, Q7: BSS138, Package_TO_SOT_SMD:SOT-23
- removed R13, R14, R17, R18, R21, R22, R25, R26: 10k, Resistor_SMD:R_0603_1608Metric_Pad0.98x0.95mm_HandSolder
- added REF**: MountingHole_2.2mm_M2_ISO14580_Pad_TopBottom, MountingHole:MountingHole_2.2mm_M2_ISO14580_Pad_TopBottom, F.Cu at (56.9, 138.4)
- added REF**: MountingHole_2.2mm_M2_ISO14580_Pad_TopBottom, MountingHole:MountingHole_2.2mm_M2_ISO14580_Pad_TopBottom, F.Cu at (149.9, 45.5)
Routing:
- added copper zone on B.Cu, net GND
- added copper zone on F.Cu, net GND
Other:
- board outline added: 100.1 x 100.1 mm

Commit message: Jack, arreglos para disipacion
Parts:
- removed REF** (x2): MountingHole_2.2mm_M2_ISO14580_Pad_TopBottom, MountingHole:MountingHole_2.2mm_M2_ISO14580_Pad_TopBottom
- J2: value USB_B_Micro -> Barrel_Jack; footprint Connector_USB:USB_Micro-B_Amphenol_10118194_Horizontal -> Connector_BarrelJack:BarrelJack_GCT_DCJ200-10-A_Horizontal
- LedVerde1: footprint Connector_JST:JST_EH_B2B-EH-A_1x02_P2.50mm_Vertical -> Connector_JST:JST_EH_S2B-EH_1x02_P2.50mm_Horizontal
- moved Q3 23.2 mm to (105.7, 108.5), turned to -90 degrees
- moved J2 6.68 mm to (63.0, 50.9)
- moved C5 5.34 mm to (71.9, 45.5)
- moved Q5 5.11 mm to (129.6, 112.3)
- moved U2 5.06 mm to (71.6, 52.3)
- moved C1 4.35 mm to (74.2, 58.9), turned to 0 degrees
Connections:
- J2 pad 2: unconnected-(J2-Pad2) -> GND
- J2 pad 3: unconnected-(J2-Pad3) -> (no net)
Routing:
- net GND: track 531.4 -> 438.8 mm
- net Net-(Bomba1-Pad1): track 56.3 -> 84.4 mm
- net /Actuadores/Conversor_NLog3/HV1: track 21.1 -> 35.5 mm
- net 5v: track 363.2 -> 372.7 mm, vias 17 -> 16
- net 3.3v: track 456.4 -> 448.8 mm
- net /Sensores/Conversor_NLog5/HV2: track 66.2 -> 59.9 mm
- net Net-(D8-Pad2): track 32.3 -> 26.1 mm
- net /Actuadores/Conversor_NLog2/HV1: track 52.8 -> 58.1 mm, vias 1 -> 2
- net Net-(10k3-Pad1): track 13.1 -> 10.9 mm
