File: CircuitDesing/embebidos/embebidos.kicad_pcb (KiCad board)
At the start: 2 copper layers, 100.1 x 100.1 mm, 84 parts, among them J1 Conn_01x03_Male, J2 Barrel_Jack, J3 Conn_01x02, Q1 BSS138, Q11 BSS138, Q13 BSS138, Q15 BSS138, Q16 BSS138, Q2 IRF540N, Q3 IRF540N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

Commit message: Codigo Agregado
Parts:
- added REF**: MountingHole_2.2mm_M2_Pad_TopBottom, MountingHole:MountingHole_2.2mm_M2_Pad_TopBottom, F.Cu at (150.4, 45.0)
- added REF**: MountingHole_2.2mm_M2_Pad_TopBottom, MountingHole:MountingHole_2.2mm_M2_Pad_TopBottom, F.Cu at (56.9, 138.9)
Routing:
- net GND: track 438.8 -> 423.9 mm
- net /Esp32Schematic/BOOT: track 51.2 -> 59.2 mm
- net 3.3v: track 448.8 -> 455.1 mm
- net Net-(Bomba1-Pad1): track 84.4 -> 80.8 mm
- net 5v: track 372.7 -> 370.2 mm, vias 16 -> 15
